File: assemble_r/assemble_r.kicad_pcb (KiCad board)
At the start: 2 copper layers, 128.5 x 102.6 mm, 51 parts, among them SW23 SW_Push, SW24 SW_Push, SW25 SW_Push, SW26 SW_Push, SW27 SW_Push, SW28 SW_Push, SW29 SW_Push, SW30 SW_Push, SW31 SW_Push, SW32 SW_Push, SW33 SW_Push, SW34 SW_Push, SW35 SW_Push, SW36 SW_Push, SW37 SW_Push, SW38 SW_Push, SW39 SW_Push, SW40 SW_Push, SW41 SW_Push, SW42 SW_Push, SW43 SW_Push, SW44 SW_SPDT, SW45 SW_Push, U23 Micon_BLEMicroPro

Commit message: feat: set prat settings
Parts:
- added Ref**: Val**, kbd_Hole:m2_Screw_Hole, F.Cu at (64.2, 117.0)
- added Ref**: Val**, kbd_Hole:m2_Screw_Hole, F.Cu at (56.7, 117.0)
Changed lines of the file:
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@@
 		(tenting front back)
 		(pcbplotparams
-			(layerselection 0x00000000_00000000_55555555_5755f5ff)
+			(layerselection 0x00000000_00000000_55555555_575555ff)
 			(plot_on_all_layers_selection 0x00000000_00000000_00000000_00000000)
 			(disableapertmacros no)
@@
 			(usegerberattributes yes)
 			(usegerberadvancedattributes yes)
-			(creategerberjobfile yes)
+			(creategerberjobfile no)
 			(dashed_line_dash_ratio 12.000000)
 			(dashed_line_gap_ratio 3.000000)
@@
 			(outputformat 1)
 			(mirror no)
-			(drillshape 1)
+			(drillshape 0)
 			(scaleselection 1)
-			(outputdirectory "")
+			(outputdirectory "../order_20250402_jcl/assemble_r")
 		)
 	)
@@
 		(embedded_fonts no)
 	)
+	(footprint "kbd_Hole:m2_Screw_Hole"
+		(layer "F.Cu")
+		(at 64.2 117)
+		(descr "Mounting Hole 2.2mm, no annular, M2")
+		(tags "mounting hole 2.2mm no annular m2")
+		(property "Reference" "Ref**"
+			(at 0 -3.2 0)
+			(layer "F.Fab")
+			(effects
+				(font
+					(size 1 1)
+					(thickness 0.15)
+				)
+			)
+		)
+		(property "Value" "Val**"
+			(at 0 3.2 0)
+			(layer "F.Fab")
+			(effects
+				(font
+					(size 1 1)
+					(thickness 0.15)
+				)
+			)
+		)
+		(property "Datasheet" ""
+			(at 0 0 0)
+			(layer "F.Fab")
+			(hide yes)
+			(effects
+				(font
+					(size 1.27 1.27)
+					(thickness 0.15)
+				)
+			)
+		)
+		(property "Description" ""
+			(at 0 0 0)
+			(layer "F.Fab")
+			(hide yes)
+			(effects
+				(font
+					(size 1.27 1.27)
+					(thickness 0.15)
+				)
+			)
+		)
+		(attr exclude_from_pos_files exclude_from_bom)
+		(fp_circle
+			(center 0 0)
+			(end 2.2 0)
+			(stroke
+				(width 0.15)
+				(type solid)
+			)
+			(fill no)
+			(layer "Cmts.User")
+		)
+		(fp_circle
+			(center 0 0)
+			(end 2.45 0)
+			(stroke
+				(width 0.05)
+				(type solid)
+			)
+			(fill no)
+			(layer "F.CrtYd")
+		)
+		(fp_text user "${REFERENCE}"
+			(at 0.3 0 0)
+			(layer "F.Fab")
+			(effects
+				(font
+					(size 1 1)
+					(thickness 0.15)
+				)
+			)
+		)
+		(pad "" np_thru_hole circle
+			(at 0 0)
+			(size 2.2 2.2)
+			(drill 2.2)
+			(layers "*.Cu" "*.Mask")
+		)
+		(embedded_fonts no)
+	)
 	(footprint "kbd_SW:Choc_v2_Hotswap_1u_16.5"
 		(layer "F.Cu")
@@
 		(embedded_fonts no)
 	)
+	(footprint "kbd_Hole:m2_Screw_Hole"
+		(layer "F.Cu")
+		(at 56.7 117)
+		(descr "Mounting Hole 2.2mm, no annular, M2")
+		(tags "mounting hole 2.2mm no annular m2")
+		(property "Reference" "Ref**"
+			(at 0 -3.2 0)
+			(layer "F.Fab")
+			(effects
+				(font
+					(size 1 1)
+					(thickness 0.15)
+				)
+			)
+		)
+		(property "Value" "Val**"
+			(at 0 3.2 0)
+			(layer "F.Fab")
+			(effects
+				(font
+					(size 1 1)
+					(thickness 0.15)
+				)
+			)
+		)
+		(property "Datasheet" ""
+			(at 0 0 0)
+			(layer "F.Fab")
+			(hide yes)
+			(effects
+				(font
+					(size 1.27 1.27)
+					(thickness 0.15)
+				)
+			)
+		)
+		(property "Description" ""
+			(at 0 0 0)
+			(layer "F.Fab")
+			(hide yes)
+			(effects
+				(font
+					(size 1.27 1.27)
+					(thickness 0.15)
+				)
+			)
+		)
+		(attr exclude_from_pos_files exclude_from_bom)
+		(fp_circle
+			(center 0 0)
+			(end 2.2 0)
+			(stroke
+				(width 0.15)
+				(type solid)
+			)
+			(fill no)
+			(layer "Cmts.User")
+		)
+		(fp_circle
+			(center 0 0)
+			(end 2.45 0)
+			(stroke
+				(width 0.05)
+				(type solid)
+			)
+			(fill no)
+			(layer "F.CrtYd")
+		)
+		(fp_text user "${REFERENCE}"
+			(at 0.3 0 0)
+			(layer "F.Fab")
+			(effects
+				(font
+					(size 1 1)
+					(thickness 0.15)
+				)
+			)
+		)
+		(pad "" np_thru_hole circle
+			(at 0 0)
+			(size 2.2 2.2)
+			(drill 2.2)
+			(layers "*.Cu" "*.Mask")
+		)
+		(embedded_fonts no)
+	)
 	(footprint "kbd_Parts:Diode_SMD"
 		(layer "F.Cu")
@@
 		)
 		(fp_line
-			(start -4.6 6.000004)
+			(start -4.6 6.000007)
 			(end -4.6 1.4)
 			(stroke
@@
 		(fp_line
 			(start -0.4 8.2)
-			(end -0.399996 3.6)
+			(end -0.399993 3.6)
 			(stroke
 				(width 0.15)
@@
 		)
 		(pad "" np_thru_hole circle
-			(at 5.000004 -5.55 2.5)
+			(at 5.000007 -5.55 2.5)
 			(size 1 1)
 			(drill oval 1)
@@
 	)
 	(segment
-		(start 52.6 122.8)
-		(end 54.4 122.8)
+		(start 54.4 122.8)
+		(end 52.6 122.8)
 		(width 0.2)
 		(layer "F.Cu")
@@
 	)
 	(segment
-		(start 52.4 90.2)
-		(end 52.4 122.6)
+		(start 51.7 121.9)
+		(end 51.7 90.2)
+		(width 0.2)
+		(layer "F.Cu")
+		(net 7)
+	)
+	(segment
+		(start 52.6 122.8)
+		(end 51.7 121.9)
 		(width 0.2)
 		(layer "F.Cu")
@@
 	)
 	(via
-		(at 52.4 90.2)
+		(at 51.7 90.2)
 		(size 0.6)
 		(drill 0.3)
@@
 		(net 7)
 	)
-	(arc
-		(start 52.4 122.6)
-		(mid 52.458579 122.741421)
-		(end 52.6 122.8)
-		(width 0.2)
-		(layer "F.Cu")
-		(net 7)
-	)
 	(segment
-		(start 48.2886 89.791)
-		(end 51.991 89.791)
+		(start 56.2 125.2)
+		(end 56.2 124.8)
 		(width 0.2)
 		(layer "B.Cu")
@@
 	)
 	(segment
-		(start 56.2 125.2)
+		(start 56.2 124.6)
 		(end 56.2 124.8)
 		(width 0.2)
@@
 	)
 	(segment
-		(start 56.2 124.6)
-		(end 56.2 124.8)
+		(start 51.7 90.2)
+		(end 51.291 89.791)
 		(width 0.2)
 		(layer "B.Cu")
@@
 	)
 	(segment
+		(start 51.291 89.791)
+		(end 48.2886 89.791)
+		(width 0.2)
+		(layer "B.Cu")
+		(net 7)
+	)
+	(segment
 		(start 90.822576 122.626689)
 		(end 78.173311 122.626689)
@@
 		(width 0.2)
 		(layer "B.Cu")
-		(net 7)
-	)
-	(arc
-		(start 51.991 89.791)
-		(mid 52.280207 89.910793)
-		(end 52.4 90.2)
-		(width 0.2)
-		(layer "B.Cu")
