File: bottom_r/bottom_r.kicad_pcb (KiCad board)
At the start: 2 copper layers, 128.5 x 102.6 mm, 4 parts

Commit message: feat: update layout
Parts:
- Ref** (x4): footprint kbd_Hole:m2_Screw_Hole -> kbd_Hole:m2_Screw_Hole_EdgeCuts
