File: middle_r/middle_r.kicad_pcb (KiCad board)
At the start: 2 copper layers, 128.5 x 102.6 mm, 0 parts

Commit message: feat: update layout
Other:
- board size 128.5 x 102.6 mm -> 128.6 x 102.6 mm
Changed lines of the file:
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@@
 	)
 	(net 0 "")
-	(gr_line
-		(start 78.365651 61.1375)
-		(end 44.965858 61.1375)
-		(stroke
-			(width 0.05)
-			(type default)
-		)
-		(layer "Edge.Cuts")
-	)
-	(gr_arc
-		(start 149.6 69.2)
-		(mid 148.892893 68.907107)
-		(end 148.6 68.2)
-		(stroke
-			(width 0.05)
-			(type default)
-		)
-		(layer "Edge.Cuts")
-	)
-	(gr_line
-		(start 143 67.6)
-		(end 144.9 67.6)
+	(gr_arc
+		(start 148 60.6)
+		(mid 148.707107 60.892893)
+		(end 149 61.6)
 		(stroke
 			(width 0.05)
@@
 	(gr_line
 		(start 167 71.1)
-		(end 145.9 71.1)
-		(stroke
-			(width 0.05)
-			(type default)
-		)
-		(layer "Edge.Cuts")
-	)
-	(gr_line
-		(start 78 67.8)
-		(end 79.7 64.6)
+		(end 146.8 71.1)
+		(stroke
+			(width 0.05)
+			(type default)
+		)
+		(layer "Edge.Cuts")
+	)
+	(gr_line
+		(start 145.8 67.6)
+		(end 145.8 70.1)
 		(stroke
 			(width 0.05)
@@
 	)
 	(gr_line
-		(start 73.2 64.6)
-		(end 48.3 64.6)
+		(start 48.3 64.6)
+		(end 73.656522 64.6)
 		(stroke
 			(width 0.05)
@@
 	)
 	(gr_line
-		(start 52.1 125.2)
-		(end 53.5 127.7)
-		(stroke
-			(width 0.05)
-			(type default)
-		)
-		(layer "Edge.Cuts")
-	)
-	(gr_arc
-		(start 43.965858 62.137707)
-		(mid 44.258682 61.430487)
-		(end 44.965858 61.1375)
+		(start 145.95 62.4)
+		(end 147.4 65.1)
 		(stroke
 			(width 0.05)
@@
 	)
 	(gr_arc
-		(start 145.9 71.1)
-		(mid 145.192893 70.807107)
-		(end 144.9 70.1)
+		(start 79.365651 59.195077)
+		(mid 79.072883 59.902059)
+		(end 78.366004 60.195077)
 		(stroke
 			(width 0.05)
@@
 	(gr_line
 		(start 139 60.6)
-		(end 147.6 60.6)
+		(end 148 60.6)
 		(stroke
 			(width 0.05)
@@
 	)
 	(gr_line
+		(start 79.3 64.6)
+		(end 78 62.4)
+		(stroke
+			(width 0.05)
+			(type default)
+		)
+		(layer "Edge.Cuts")
+	)
+	(gr_line
 		(start 110 136.802009)
 		(end 110 126.999389)
@@
 		(layer "Edge.Cuts")
 	)
-	(gr_arc
-		(start 79.365651 60.1375)
-		(mid 79.072755 60.844589)
-		(end 78.365651 61.1375)
+	(gr_line
+		(start 78 62.4)
+		(end 74.9 62.4)
 		(stroke
 			(width 0.05)
@@
 		(start 120.6 121.1)
 		(end 121.8 123.3)
-		(stroke
-			(width 0.05)
-			(type default)
-		)
-		(layer "Edge.Cuts")
-	)
-	(gr_line
-		(start 141.4 64.7)
-		(end 143 67.6)
 		(stroke
 			(width 0.05)
@@
 	)
 	(gr_line
-		(start 73.2 64.6)
-		(end 75 67.8)
-		(stroke
-			(width 0.05)
-			(type default)
-		)
-		(layer "Edge.Cuts")
-	)
-	(gr_line
-		(start 51.012616 132.295892)
-		(end 55.518819 146.136372)
+		(start 74.9 62.4)
+		(end 73.656522 64.6)
+		(stroke
+			(width 0.05)
+			(type default)
+		)
+		(layer "Edge.Cuts")
+	)
+	(gr_line
+		(start 48.710265 125.196708)
+		(end 47.7 127.9)
+		(stroke
+			(width 0.05)
+			(type default)
+		)
+		(layer "Edge.Cuts")
+	)
+	(gr_line
+		(start 79.7 64.6)
+		(end 79.3 64.6)
+		(stroke
+			(width 0.05)
+			(type default)
+		)
+		(layer "Edge.Cuts")
+	)
+	(gr_line
+		(start 55.518819 146.136372)
+		(end 50.427907 130.5)
 		(stroke
 			(width 0.05)
@@
 	)
 	(gr_line
+		(start 142.65 62.4)
+		(end 145.95 62.4)
+		(stroke
+			(width 0.05)
+			(type default)
+		)
+		(layer "Edge.Cuts")
+	)
+	(gr_line
 		(start 79.365651 48.737079)
-		(end 79.365651 60.1375)
+		(end 79.365651 59.195077)
 		(stroke
 			(width 0.05)
@@
 		(start 47.3 120.8)
 		(end 48.710265 125.196708)
-		(stroke
-			(width 0.05)
-			(type default)
-		)
-		(layer "Edge.Cuts")
-	)
-	(gr_line
-		(start 148.6 61.6)
-		(end 148.6 68.2)
 		(stroke
 			(width 0.05)
@@
 	)
 	(gr_line
-		(start 75 67.8)
-		(end 78 67.8)
-		(stroke
-			(width 0.05)
-			(type default)
-		)
-		(layer "Edge.Cuts")
-	)
-	(gr_line
 		(start 82.4 64.6)
 		(end 79.7 64.6)
@@
 	)
 	(gr_line
+		(start 44.856952 60.206909)
+		(end 78.366004 60.195077)
+		(stroke
+			(width 0.05)
+			(type default)
+		)
+		(layer "Edge.Cuts")
+	)
+	(gr_line
 		(start 134.1 51.8)
 		(end 84.4 51.8)
@@
 		(layer "Edge.Cuts")
 	)
-	(gr_arc
-		(start 44.025412 121.610664)
-		(mid 43.990032 121.46065)
-		(end 43.978119 121.306981)
+	(gr_line
+		(start 47.7 127.9)
+		(end 49 130.5)
 		(stroke
 			(width 0.05)
@@
 	)
 	(gr_line
-		(start 53.5 127.7)
-		(end 51.012616 132.295892)
+		(start 141.4 64.7)
+		(end 142.65 62.4)
 		(stroke
 			(width 0.05)
@@
 	)
 	(gr_line
-		(start 48.710265 125.196708)
-		(end 52.1 125.2)
-		(stroke
-			(width 0.05)
-			(type default)
-		)
-		(layer "Edge.Cuts")
-	)
-	(gr_line
-		(start 149.6 69.2)
+		(start 150 69.2)
 		(end 171.401401 69.2)
 		(stroke
@@
 	)
 	(gr_line
-		(start 44.025412 121.610664)
+		(start 43.869771 121.364243)
 		(end 52.959724 149.62005)
 		(stroke
@@
 	)
 	(gr_line
-		(start 43.965858 62.137707)
-		(end 43.978119 121.306981)
-		(stroke
-			(width 0.05)
-			(type default)
-		)
-		(layer "Edge.Cuts")
-	)
-	(gr_arc
-		(start 147.6 60.6)
-		(mid 148.307107 60.892893)
-		(end 148.6 61.6)
+		(start 43.857305 61.207116)
+		(end 43.869771 121.364243)
+		(stroke
+			(width 0.05)
+			(type default)
+		)
+		(layer "Edge.Cuts")
+	)
+	(gr_arc
+		(start 146.8 71.1)
+		(mid 146.092893 70.807107)
+		(end 145.8 70.1)
 		(stroke
 			(width 0.05)
@@
 	)
 	(gr_line
-		(start 144.9 70.1)
-		(end 144.9 67.6)
+		(start 149 61.6)
+		(end 149 68.2)
+		(stroke
+			(width 0.05)
+			(type default)
+		)
+		(layer "Edge.Cuts")
+	)
+	(gr_line
+		(start 49 130.5)
+		(end 50.427907 130.5)
 		(stroke
 			(width 0.05)
@@
 		(start 141.4 64.7)
 		(end 136.1 64.7)
+		(stroke
+			(width 0.05)
+			(type default)
+		)
+		(layer "Edge.Cuts")
+	)
+	(gr_line
+		(start 147.4 65.1)
+		(end 145.8 67.6)
+		(stroke
+			(width 0.05)
+			(type default)
+		)
+		(layer "Edge.Cuts")
+	)
+	(gr_arc
+		(start 150 69.2)
+		(mid 149.292893 68.907107)
+		(end 149 68.2)
 		(stroke
 			(width 0.05)
@@
 		(stroke
 			(width 0.05)
+			(type default)
+		)
+		(layer "Edge.Cuts")
+	)
+	(gr_arc
+		(start 43.857305 61.207116)
+		(mid 44.15 60.5)
+		(end 44.856952 60.206909)
+		(stroke
+			(width 0.05)
